File: Nico Ortho.kicad_pcb (KiCad board)
At the start: 2 copper layers, 62 parts, among them SW10 SW_PUSH, SW11 SW_PUSH, SW12 SW_PUSH, SW13 SW_PUSH, SW14 SW_PUSH, SW15 SW_PUSH, SW16 SW_PUSH, SW17 SW_PUSH, SW18 SW_PUSH, SW19 SW_PUSH, SW20 SW_PUSH, SW21 SW_PUSH, SW22 SW_PUSH, SW23 SW_PUSH, SW24 SW_PUSH, SW25 SW_PUSH, SW26 SW_PUSH, SW27 SW_PUSH, SW28 SW_PUSH, SW29 SW_PUSH, SW30 SW_PUSH, SW6 SW_PUSH, SW7 SW_PUSH, SW8 SW_PUSH, SW9 SW_PUSH

Commit message: Checkpoint
Parts:
- removed D1, D10, D11, D12, D13, D14, D15, D16, D17, D18, D19, D2, D20, D21, D22, D23, D24, D25, D3, D4, D5, D6, D7, D8, D9: D, kbd:D3_TH_SMD
- removed the REFr at (152.0, 49.5)
- removed the REFr1 at (152.0, 52.0)
- removed the REFr2 at (152.0, 54.6)
- removed the REFr3 at (152.0, 57.1)
- removed the REFr4 at (152.0, 59.7)
- removed the SW6 at (64.5, 121.0)
- removed the SW6 at (55.0, 45.0)
- added D33: D, kbd:D3_TH_SMD_v2, F.Cu at (64.3, 42.7)
- added D34: D, kbd:D3_TH_SMD_v2, F.Cu at (83.3, 42.7)
- added D35: D, kbd:D3_TH_SMD_v2, F.Cu at (102.3, 42.7)
- added D36: D, kbd:D3_TH_SMD_v2, F.Cu at (121.3, 42.7)
- added D37: D, kbd:D3_TH_SMD_v2, F.Cu at (140.3, 42.7)
- added D38: D, kbd:D3_TH_SMD_v2, F.Cu at (64.3, 61.7)
- added D39: D, kbd:D3_TH_SMD_v2, F.Cu at (83.3, 61.7)
- added D40: D, kbd:D3_TH_SMD_v2, F.Cu at (102.3, 61.7)
- added D41: D, kbd:D3_TH_SMD_v2, F.Cu at (121.3, 61.7)
- added D42: D, kbd:D3_TH_SMD_v2, F.Cu at (140.3, 61.7)
- added D43: D, kbd:D3_TH_SMD_v2, F.Cu at (64.3, 80.7)
- added D44: D, kbd:D3_TH_SMD_v2, F.Cu at (83.3, 80.7)
- added D45: D, kbd:D3_TH_SMD_v2, F.Cu at (102.3, 80.7)
- added D46: D, kbd:D3_TH_SMD_v2, F.Cu at (121.3, 80.7)
- added D47: D, kbd:D3_TH_SMD_v2, F.Cu at (140.3, 80.7)
- added D48: D, kbd:D3_TH_SMD_v2, F.Cu at (64.3, 99.7)
- added D49: D, kbd:D3_TH_SMD_v2, F.Cu at (83.3, 99.7)
- added D50: D, kbd:D3_TH_SMD_v2, F.Cu at (102.3, 99.7)
- added D51: D, kbd:D3_TH_SMD_v2, F.Cu at (121.3, 99.7)
- added D52: D, kbd:D3_TH_SMD_v2, F.Cu at (140.3, 99.7)
- added D53: D, kbd:D3_TH_SMD_v2, F.Cu at (64.3, 118.7)
- added D54: D, kbd:D3_TH_SMD_v2, F.Cu at (83.3, 118.7)
- added D55: D, kbd:D3_TH_SMD_v2, F.Cu at (102.3, 118.7)
- added D56: D, kbd:D3_TH_SMD_v2, F.Cu at (121.3, 118.7)
- added D57: D, kbd:D3_TH_SMD_v2, F.Cu at (140.3, 118.7)
- added REFr: SolderWire-0.1sqmm_1x01_D0.4mm_OD1mm, Connector_Wire:SolderWire-0.1sqmm_1x01_D0.4mm_OD1mm, F.Cu at (53.5, 48.9)
- added REFr: SolderWire-0.1sqmm_1x01_D0.4mm_OD1mm, Connector_Wire:SolderWire-0.1sqmm_1x01_D0.4mm_OD1mm, F.Cu at (-25.0, 22.3)
- added REFr1: SolderWire-0.1sqmm_1x01_D0.4mm_OD1mm, Connector_Wire:SolderWire-0.1sqmm_1x01_D0.4mm_OD1mm, F.Cu at (-25.0, 24.8)
- added REFr1: SolderWire-0.1sqmm_1x01_D0.4mm_OD1mm, Connector_Wire:SolderWire-0.1sqmm_1x01_D0.4mm_OD1mm, F.Cu at (53.5, 51.4)
- added REFr10: SolderWire-0.1sqmm_1x01_D0.4mm_OD1mm, Connector_Wire:SolderWire-0.1sqmm_1x01_D0.4mm_OD1mm, F.Cu at (146.0, 87.0)
- added REFr10: SolderWire-0.1sqmm_1x01_D0.4mm_OD1mm, Connector_Wire:SolderWire-0.1sqmm_1x01_D0.4mm_OD1mm, F.Cu at (146.0, 121.4)
- added REFr11: SolderWire-0.1sqmm_1x01_D0.4mm_OD1mm, Connector_Wire:SolderWire-0.1sqmm_1x01_D0.4mm_OD1mm, F.Cu at (146.0, 124.0)
- added REFr11: SolderWire-0.1sqmm_1x01_D0.4mm_OD1mm, Connector_Wire:SolderWire-0.1sqmm_1x01_D0.4mm_OD1mm, F.Cu at (146.0, 89.5)
- added REFr12: SolderWire-0.1sqmm_1x01_D0.4mm_OD1mm, Connector_Wire:SolderWire-0.1sqmm_1x01_D0.4mm_OD1mm, F.Cu at (146.0, 126.5)
- added REFr12: SolderWire-0.1sqmm_1x01_D0.4mm_OD1mm, Connector_Wire:SolderWire-0.1sqmm_1x01_D0.4mm_OD1mm, F.Cu at (146.0, 92.1)
- added REFr13: SolderWire-0.1sqmm_1x01_D0.4mm_OD1mm, Connector_Wire:SolderWire-0.1sqmm_1x01_D0.4mm_OD1mm, F.Cu at (146.0, 129.1)
- added REFr13: SolderWire-0.1sqmm_1x01_D0.4mm_OD1mm, Connector_Wire:SolderWire-0.1sqmm_1x01_D0.4mm_OD1mm, F.Cu at (146.0, 94.6)
- added REFr14: SolderWire-0.1sqmm_1x01_D0.4mm_OD1mm, Connector_Wire:SolderWire-0.1sqmm_1x01_D0.4mm_OD1mm, F.Cu at (146.0, 131.6)
- added REFr14: SolderWire-0.1sqmm_1x01_D0.4mm_OD1mm, Connector_Wire:SolderWire-0.1sqmm_1x01_D0.4mm_OD1mm, F.Cu at (146.0, 97.1)
- added REFr2: SolderWire-0.1sqmm_1x01_D0.4mm_OD1mm, Connector_Wire:SolderWire-0.1sqmm_1x01_D0.4mm_OD1mm, F.Cu at (-25.0, 27.4)
- added REFr2: SolderWire-0.1sqmm_1x01_D0.4mm_OD1mm, Connector_Wire:SolderWire-0.1sqmm_1x01_D0.4mm_OD1mm, F.Cu at (53.5, 54.0)
- added REFr3: SolderWire-0.1sqmm_1x01_D0.4mm_OD1mm, Connector_Wire:SolderWire-0.1sqmm_1x01_D0.4mm_OD1mm, F.Cu at (53.5, 56.5)
- added REFr3: SolderWire-0.1sqmm_1x01_D0.4mm_OD1mm, Connector_Wire:SolderWire-0.1sqmm_1x01_D0.4mm_OD1mm, F.Cu at (-25.0, 29.9)
- added REFr4: SolderWire-0.1sqmm_1x01_D0.4mm_OD1mm, Connector_Wire:SolderWire-0.1sqmm_1x01_D0.4mm_OD1mm, F.Cu at (53.5, 59.0)
- added REFr4: SolderWire-0.1sqmm_1x01_D0.4mm_OD1mm, Connector_Wire:SolderWire-0.1sqmm_1x01_D0.4mm_OD1mm, F.Cu at (-25.0, 32.5)
- added REFr5: SolderWire-0.1sqmm_1x01_D0.4mm_OD1mm, Connector_Wire:SolderWire-0.1sqmm_1x01_D0.4mm_OD1mm, F.Cu at (53.5, 87.0)
- added REFr5: SolderWire-0.1sqmm_1x01_D0.4mm_OD1mm, Connector_Wire:SolderWire-0.1sqmm_1x01_D0.4mm_OD1mm, F.Cu at (53.5, 121.4)
- added REFr5: SolderWire-0.1sqmm_1x01_D0.4mm_OD1mm, Connector_Wire:SolderWire-0.1sqmm_1x01_D0.4mm_OD1mm, F.Cu at (146.0, 48.9)
- added REFr6: SolderWire-0.1sqmm_1x01_D0.4mm_OD1mm, Connector_Wire:SolderWire-0.1sqmm_1x01_D0.4mm_OD1mm, F.Cu at (146.0, 51.4)
- added REFr6: SolderWire-0.1sqmm_1x01_D0.4mm_OD1mm, Connector_Wire:SolderWire-0.1sqmm_1x01_D0.4mm_OD1mm, F.Cu at (53.5, 124.0)
- added REFr6: SolderWire-0.1sqmm_1x01_D0.4mm_OD1mm, Connector_Wire:SolderWire-0.1sqmm_1x01_D0.4mm_OD1mm, F.Cu at (53.5, 89.5)
- added REFr7: SolderWire-0.1sqmm_1x01_D0.4mm_OD1mm, Connector_Wire:SolderWire-0.1sqmm_1x01_D0.4mm_OD1mm, F.Cu at (146.0, 54.0)
- added REFr7: SolderWire-0.1sqmm_1x01_D0.4mm_OD1mm, Connector_Wire:SolderWire-0.1sqmm_1x01_D0.4mm_OD1mm, F.Cu at (53.5, 126.5)
- added REFr7: SolderWire-0.1sqmm_1x01_D0.4mm_OD1mm, Connector_Wire:SolderWire-0.1sqmm_1x01_D0.4mm_OD1mm, F.Cu at (53.5, 92.1)
- added REFr8: SolderWire-0.1sqmm_1x01_D0.4mm_OD1mm, Connector_Wire:SolderWire-0.1sqmm_1x01_D0.4mm_OD1mm, F.Cu at (53.5, 129.1)
- added REFr8: SolderWire-0.1sqmm_1x01_D0.4mm_OD1mm, Connector_Wire:SolderWire-0.1sqmm_1x01_D0.4mm_OD1mm, F.Cu at (146.0, 56.5)
- added REFr8: SolderWire-0.1sqmm_1x01_D0.4mm_OD1mm, Connector_Wire:SolderWire-0.1sqmm_1x01_D0.4mm_OD1mm, F.Cu at (53.5, 94.6)
- added REFr9: SolderWire-0.1sqmm_1x01_D0.4mm_OD1mm, Connector_Wire:SolderWire-0.1sqmm_1x01_D0.4mm_OD1mm, F.Cu at (146.0, 59.0)
- added REFr9: SolderWire-0.1sqmm_1x01_D0.4mm_OD1mm, Connector_Wire:SolderWire-0.1sqmm_1x01_D0.4mm_OD1mm, F.Cu at (53.5, 131.6)
- added REFr9: SolderWire-0.1sqmm_1x01_D0.4mm_OD1mm, Connector_Wire:SolderWire-0.1sqmm_1x01_D0.4mm_OD1mm, F.Cu at (53.5, 97.1)
- added SW6: SW_PUSH, kbd:CherryMX_1u, F.Cu at (61.7, 50.9)
- moved SW11 8.93 mm to (61.7, 69.9)
- moved SW12 8.93 mm to (80.7, 69.9)
- moved SW13 8.93 mm to (99.7, 69.9)
- moved SW14 8.93 mm to (118.7, 69.9)
- moved SW16 8.93 mm to (61.7, 88.9)
- moved SW17 8.93 mm to (80.7, 88.9)
- moved SW18 8.93 mm to (99.7, 88.9)
- moved SW19 8.93 mm to (118.7, 88.9)
- moved SW21 8.93 mm to (61.7, 107.9)
- moved SW22 8.93 mm to (80.7, 107.9)
- moved SW23 8.93 mm to (99.7, 107.9)
- moved SW24 8.93 mm to (118.7, 107.9)
- moved SW26 8.93 mm to (61.7, 126.9)
- moved SW27 8.93 mm to (80.7, 126.9)
- moved SW28 8.93 mm to (99.7, 126.9)
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Routing:
- net (no net): track 900.3 -> 176.8 mm

Commit message: Checkpoint
Parts:
- removed the REFr at (26.5, 60.0)
- removed the REFr at (28.5, 48.0)
- removed the REFr at (-25.0, 22.3)
- removed the REFr1 at (-25.0, 24.8)
- removed the REFr1 at (26.5, 62.5)
- removed the REFr2 at (-25.0, 27.4)
- removed the REFr2 at (26.5, 65.1)
- removed the REFr3 at (26.5, 67.6)
- removed the REFr3 at (-25.0, 29.9)
- removed the REFr4 at (26.5, 70.2)
- removed the REFr4 at (-25.0, 32.5)
Routing:
- net (no net): track 176.8 -> 556.8 mm

Commit message: Checkpoint
Connections:
- SW10 pad 2: (no net) -> col5
- SW11 pad 2: (no net) -> col1
- SW12 pad 2: (no net) -> col2
- SW13 pad 2: (no net) -> col3
- SW14 pad 2: (no net) -> col4
- SW15 pad 2: (no net) -> col5
- SW16 pad 2: (no net) -> col1
- SW17 pad 2: (no net) -> col2
- SW18 pad 2: (no net) -> col3
- SW19 pad 2: (no net) -> col4
- SW20 pad 2: (no net) -> col5
- SW21 pad 2: (no net) -> col1
- SW22 pad 2: (no net) -> col2
- SW23 pad 2: (no net) -> col3
- SW24 pad 2: (no net) -> col4
- SW25 pad 2: (no net) -> col5
- SW26 pad 2: (no net) -> col1
- SW27 pad 2: (no net) -> col2
- SW28 pad 2: (no net) -> col3
- SW29 pad 2: (no net) -> col4
- SW30 pad 2: (no net) -> col5
- SW6 pad 2: (no net) -> col1
- SW7 pad 2: (no net) -> col2
- SW8 pad 2: (no net) -> col3
- SW9 pad 2: (no net) -> col4
Routing:
- net (no net): track 556.8 -> 699.9 mm
- net col5: track 0.00 -> 76.0 mm
- net col4: track 0.00 -> 76.0 mm
- net col3: track 0.00 -> 76.0 mm
- net col2: track 0.00 -> 76.0 mm
- net col1: track 0.00 -> 76.0 mm

Commit message: Checkpoint
Connections:
- D38 pad 1: (no net) -> row2
- D39 pad 1: (no net) -> row2
- D40 pad 1: (no net) -> row2
- D41 pad 1: (no net) -> row2
- D42 pad 1: (no net) -> row2
- D43 pad 1: (no net) -> row3
- D44 pad 1: (no net) -> row3
- D45 pad 1: (no net) -> row3
- D46 pad 1: (no net) -> row3
- D47 pad 1: (no net) -> row3
- D48 pad 1: (no net) -> row4
- D49 pad 1: (no net) -> row4
- D50 pad 1: (no net) -> row4
- D51 pad 1: (no net) -> row4
- D52 pad 1: (no net) -> row4
- D53 pad 1: (no net) -> row5
- D54 pad 1: (no net) -> row5
- D55 pad 1: (no net) -> row5
- D56 pad 1: (no net) -> row5
- D57 pad 1: (no net) -> row5
- REFr10 pad 1: (no net) -> row3
- REFr10 pad 1: (no net) -> row5
- REFr14 pad 1: (no net) -> row4
- REFr4 pad 1: (no net) -> row2
- REFr5 pad 1: (no net) -> row3
- REFr5 pad 1: (no net) -> row5
- REFr9 pad 1: (no net) -> row2
- REFr9 pad 1: (no net) -> row4
Routing:
- net (no net): track 699.9 -> 282.7 mm
- net row3: track 0.00 -> 109.5 mm
- net row4: track 0.00 -> 104.3 mm
- net row5: track 0.00 -> 102.2 mm
- net row2: track 0.00 -> 101.1 mm

Commit message: Checkpoint
Parts:
- added SW6: SW_PUSH, kbd:CherryMX_1u, F.Cu at (71.2, 126.9)
Connections:
- D33 pad 1: (no net) -> row1
- D34 pad 1: (no net) -> row1
- D35 pad 1: (no net) -> row1
- D36 pad 1: (no net) -> row1
- D37 pad 1: (no net) -> row1
- REFr pad 1: (no net) -> row1
- REFr5 pad 1: (no net) -> row1
Routing:
- net row1: track 0.00 -> 105.9 mm
- net (no net): track 282.7 -> 186.3 mm
- net col2: track 76.0 -> 85.5 mm

Commit message: Checkpoint
Parts:
- added REF**: PinHeader_1x04_P2.54mm_Vertical, Connector_PinHeader_2.54mm:PinHeader_1x04_P2.54mm_Vertical, F.Cu at (70.0, 42.7)
- added REF**1: PinHeader_1x04_P2.54mm_Vertical, Connector_PinHeader_2.54mm:PinHeader_1x04_P2.54mm_Vertical, F.Cu at (89.0, 42.7)
- added REF**2: PinHeader_1x04_P2.54mm_Vertical, Connector_PinHeader_2.54mm:PinHeader_1x04_P2.54mm_Vertical, F.Cu at (108.0, 42.7)
- added REF**3: PinHeader_1x04_P2.54mm_Vertical, Connector_PinHeader_2.54mm:PinHeader_1x04_P2.54mm_Vertical, F.Cu at (127.0, 42.7)
Routing:
- net row5: track 102.2 -> 181.4 mm
- net row4: track 104.3 -> 165.6 mm
- net row3: track 109.5 -> 150.7 mm
- net row2: track 101.1 -> 122.3 mm
- net col5: track 76.0 -> 96.5 mm
- net col4: track 76.0 -> 83.1 mm
- net col3: track 76.0 -> 83.1 mm
- net col2: track 85.5 -> 92.6 mm
- net col1: track 76.0 -> 83.1 mm
- net row1: track 105.9 -> 107.9 mm

Commit message: Checkpoint
Other:
- board outline added: 95 x 95 mm
- board text added: "col1"
- board text added: "col2"
- board text added: "col3"
- board text added: "col4"
- board text added: "col5"
- board text added: "row1"
- board text added: "row2"
- board text added: "row3"
- board text added: "row4"
- board text added: "row5"
Changed lines of the file:
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@@
     )
+  )
+  (gr_line (start 52.25 136.39) (end 147.25 136.39) (layer "Edge.Cuts") (width 0.05))
+  (gr_line (start 52.25 41.39) (end 52.25 136.39) (layer "Edge.Cuts") (width 0.05))
+  (gr_line (start 147.25 136.39) (end 147.25 41.39) (layer "Edge.Cuts") (width 0.05))
+  (gr_line (start 147.25 41.39) (end 52.25 41.39) (layer "Edge.Cuts") (width 0.05))
+  (gr_text "col5" (at 129.4 45.4 90) (layer "B.SilkS")
+    (effects (font (size 1 1) (thickness 0.15)) (justify mirror))
+  )
+  (gr_text "row5" (at 142.7 120.3) (layer "B.SilkS")
+    (effects (font (size 1 1) (thickness 0.15)) (justify mirror))
+  )
+  (gr_text "row2" (at 56.3 59.1) (layer "B.SilkS")
+    (effects (font (size 1 1) (thickness 0.15)) (justify mirror))
+  )
+  (gr_text "col2" (at 88.7 45.6 90) (layer "B.SilkS")
+    (effects (font (size 1 1) (thickness 0.15)) (justify mirror))
+  )
+  (gr_text "row1" (at 145.1 47.1) (layer "B.SilkS")
+    (effects (font (size 1 1) (thickness 0.15)) (justify mirror))
+  )
+  (gr_text "row2" (at 72.3 45.6 90) (layer "B.SilkS")
+    (effects (font (size 1 1) (thickness 0.15)) (justify mirror))
+  )
+  (gr_text "row3" (at 145.1 84.9) (layer "B.SilkS")
+    (effects (font (size 1 1) (thickness 0.15)) (justify mirror))
+  )
+  (gr_text "row2" (at 142.9 59.2) (layer "B.SilkS")
+    (effects (font (size 1 1) (thickness 0.15)) (justify mirror))
+  )
+  (gr_text "col1" (at 70 45.6 90) (layer "B.SilkS")
+    (effects (font (size 1 1) (thickness 0.15)) (justify mirror))
+  )
+  (gr_text "row4" (at 142.9 97.3) (layer "B.SilkS")
+    (effects (font (size 1 1) (thickness 0.15)) (justify mirror))
+  )
+  (gr_text "row4" (at 56.8 97.2) (layer "B.SilkS")
+    (effects (font (size 1 1) (thickness 0.15)) (justify mirror))
+  )
+  (gr_text "col4" (at 126.8 45.4 90) (layer "B.SilkS")
+    (effects (font (size 1 1) (thickness 0.15)) (justify mirror))
+  )
+  (gr_text "row5" (at 94.1 45.3 90) (layer "B.SilkS")
+    (effects (font (size 1 1) (thickness 0.15)) (justify mirror))
+  )
+  (gr_text "row3" (at 74.9 45.6 90) (layer "B.SilkS")
+    (effects (font (size 1 1) (thickness 0.15)) (justify mirror))
+  )
+  (gr_text "col3" (at 107.9 45.3 90) (layer "B.SilkS")
+    (effects (font (size 1 1) (thickness 0.15)) (justify mirror))
+  )
+  (gr_text "row4" (at 77.4 45.5 90) (layer "B.SilkS")
+    (effects (font (size 1 1) (thickness 0.15)) (justify mirror))
+  )
+  (gr_text "row1" (at 54.8 47.1) (layer "B.SilkS")
+    (effects (font (size 1 1) (thickness 0.15)) (justify mirror))
+  )
+  (gr_text "row3" (at 54.4 85) (layer "B.SilkS")
+    (effects (font (size 1 1) (thickness 0.15)) (justify mirror))
+  )
+  (gr_text "row5" (at 56.4 121.3) (layer "B.SilkS")
+    (effects (font (size 1 1) (thickness 0.15)) (justify mirror))
+  )
+  (gr_text "row1" (at 91.5 45.3 90) (layer "B.SilkS")
+    (effects (font (size 1 1) (thickness 0.15)) (justify mirror))
   )
   (segment (start 67.39 124.36) (end 76.89 124.36) (width 0.25) (layer "F.Cu") (net 0))
